File: Buck_Boost_Controller/Buck_Boost_Controller/Buck_Boost_Controller.kicad_sch (KiCad schematic)
At the start: 15 parts, among them U1 BQ25858QWRRVRQ1, U2 CSD19506KTT, U3 CSD19506KTT, U4 CSD19506KTT, U5 CSD19506KTT

Commit message: Update Buck_Boost_Controller.kicad_sch
Other:
- note added: "Buck-Boost Controller"
- moved on the sheet: R5, U1
