File: LV_Regulator/mcu.kicad_sch (KiCad schematic)
At the start: 14 parts, among them U2 STM32F103C8Tx

Commit message: Fixed last commit
Fixed all mistakes from the last push
Connections:
- net VDDA is gone; now on net +3V3: C11.1, C12.1, U2.9 (VDDA)
Changed lines of the file:
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@@
 	)
 	(junction
+		(at 204.47 40.64)
+		(diameter 0)
+		(color 0 0 0 0)
+	)
+	(junction
 		(at 212.09 26.67)
 		(diameter 0)
@@
 	)
 	(symbol
+		(lib_id "power:+3V3")
+		(at 205.74 54.61 0)
+		(unit 1)
+		(exclude_from_sim no)
+		(in_bom yes)
+		(on_board yes)
+		(dnp no)
+		(fields_autoplaced yes)
+		(property "Reference" "#PWR065"
+			(at 205.74 58.42 0)
+			(effects
+				(font
+					(size 1.27 1.27)
+				)
+				(hide yes)
+			)
+		)
+		(property "Value" "+3V3"
+			(at 205.74 49.53 0)
+			(effects
+				(font
+					(size 1.27 1.27)
+				)
+			)
+		)
+		(property "Footprint" ""
+			(at 205.74 54.61 0)
+			(effects
+				(font
+					(size 1.27 1.27)
+				)
+				(hide yes)
+			)
+		)
+		(property "Datasheet" ""
+			(at 205.74 54.61 0)
+			(effects
+				(font
+					(size 1.27 1.27)
+				)
+				(hide yes)
+			)
+		)
+		(property "Description" "Power symbol creates a global label with name \"+3V3\""
+			(at 205.74 54.61 0)
+			(effects
+				(font
+					(size 1.27 1.27)
+				)
+				(hide yes)
+			)
+		)
+		(pin "1"
+		)
+		(instances
+			(project "LV_Regulator"
+				(path "/9003ce10-3354-47c9-924a-fd038a206791/7dabe8d0-f22d-4d1e-a460-c5fc9599efb1"
+					(reference "#PWR065")
+					(unit 1)
+				)
+			)
+		)
+	)
+	(symbol
 		(lib_id "Jumper:SolderJumper_3_Open")
 		(at 158.75 24.13 90)
@@
 					(unit 1)
 				)
-				(path "/9003ce10-3354-47c9-924a-fd038a206791/7dfce8f1-0c22-480c-91d4-3ffb0e2b2dff"
-					(reference "JP9")
-					(unit 1)
-				)
 			)
 		)
@@
 					(unit 1)
 				)
-				(path "/9003ce10-3354-47c9-924a-fd038a206791/7dfce8f1-0c22-480c-91d4-3ffb0e2b2dff"
-					(reference "JP7")
-					(unit 1)
-				)
 			)
 		)
@@
 					(unit 1)
 				)
-				(path "/9003ce10-3354-47c9-924a-fd038a206791/7dfce8f1-0c22-480c-91d4-3ffb0e2b2dff"
-					(reference "#PWR064")
-					(unit 1)
-				)
 			)
 		)
@@
 					(unit 1)
 				)
-				(path "/9003ce10-3354-47c9-924a-fd038a206791/7dfce8f1-0c22-480c-91d4-3ffb0e2b2dff"
-					(reference "#PWR067")
-					(unit 1)
-				)
 			)
 		)
@@
 					(unit 1)
 				)
-				(path "/9003ce10-3354-47c9-924a-fd038a206791/7dfce8f1-0c22-480c-91d4-3ffb0e2b2dff"
-					(reference "C23")
-					(unit 1)
-				)
 			)
 		)
@@
 					(unit 1)
 				)
-				(path "/9003ce10-3354-47c9-924a-fd038a206791/7dfce8f1-0c22-480c-91d4-3ffb0e2b2dff"
-					(reference "JP12")
-					(unit 1)
-				)
 			)
 		)
@@
 					(unit 1)
 				)
-				(path "/9003ce10-3354-47c9-924a-fd038a206791/7dfce8f1-0c22-480c-91d4-3ffb0e2b2dff"
-					(reference "C24")
-					(unit 1)
-				)
 			)
 		)
@@
 					(unit 1)
 				)
-				(path "/9003ce10-3354-47c9-924a-fd038a206791/7dfce8f1-0c22-480c-91d4-3ffb0e2b2dff"
-					(reference "C21")
-					(unit 1)
-				)
 			)
 		)
@@
 					(unit 1)
 				)
-				(path "/9003ce10-3354-47c9-924a-fd038a206791/7dfce8f1-0c22-480c-91d4-3ffb0e2b2dff"
-					(reference "C22")
-					(unit 1)
-				)
 			)
 		)
@@
 					(unit 1)
 				)
-				(path "/9003ce10-3354-47c9-924a-fd038a206791/7dfce8f1-0c22-480c-91d4-3ffb0e2b2dff"
-					(reference "#PWR066")
-					(unit 1)
-				)
 			)
 		)
@@
 					(unit 1)
 				)
-				(path "/9003ce10-3354-47c9-924a-fd038a206791/7dfce8f1-0c22-480c-91d4-3ffb0e2b2dff"
-					(reference "#PWR072")
-					(unit 1)
-				)
 			)
 		)
@@
 					(unit 1)
 				)
-				(path "/9003ce10-3354-47c9-924a-fd038a206791/7dfce8f1-0c22-480c-91d4-3ffb0e2b2dff"
-					(reference "C25")
-					(unit 1)
-				)
 			)
 		)
@@
 					(unit 1)
 				)
-				(path "/9003ce10-3354-47c9-924a-fd038a206791/7dfce8f1-0c22-480c-91d4-3ffb0e2b2dff"
-					(reference "#PWR060")
-					(unit 1)
-				)
 			)
 		)
@@
 					(unit 1)
 				)
-				(path "/9003ce10-3354-47c9-924a-fd038a206791/7dfce8f1-0c22-480c-91d4-3ffb0e2b2dff"
-					(reference "#PWR069")
-					(unit 1)
-				)
 			)
 		)
@@
 					(unit 1)
 				)
-				(path "/9003ce10-3354-47c9-924a-fd038a206791/7dfce8f1-0c22-480c-91d4-3ffb0e2b2dff"
-					(reference "#PWR059")
-					(unit 1)
-				)
 			)
 		)
@@
 					(unit 1)
 				)
-				(path "/9003ce10-3354-47c9-924a-fd038a206791/7dfce8f1-0c22-480c-91d4-3ffb0e2b2dff"
-					(reference "JP11")
-					(unit 1)
-				)
 			)
 		)
@@
 					(unit 1)
 				)
-				(path "/9003ce10-3354-47c9-924a-fd038a206791/7dfce8f1-0c22-480c-91d4-3ffb0e2b2dff"
-					(reference "#PWR062")
-					(unit 1)
-				)
 			)
 		)
@@
 					(unit 1)
 				)
-				(path "/9003ce10-3354-47c9-924a-fd038a206791/7dfce8f1-0c22-480c-91d4-3ffb0e2b2dff"
-					(reference "#PWR074")
-					(unit 1)
-				)
 			)
 		)
@@
 					(unit 1)
 				)
-				(path "/9003ce10-3354-47c9-924a-fd038a206791/7dfce8f1-0c22-480c-91d4-3ffb0e2b2dff"
-					(reference "JP8")
-					(unit 1)
-				)
 			)
 		)
@@
 					(unit 1)
 				)
-				(path "/9003ce10-3354-47c9-924a-fd038a206791/7dfce8f1-0c22-480c-91d4-3ffb0e2b2dff"
-					(reference "C20")
-					(unit 1)
-				)
 			)
 		)
@@
 					(unit 1)
 				)
-				(path "/9003ce10-3354-47c9-924a-fd038a206791/7dfce8f1-0c22-480c-91d4-3ffb0e2b2dff"
-					(reference "#PWR070")
-					(unit 1)
-				)
 			)
 		)
@@
 					(unit 1)
 				)
-				(path "/9003ce10-3354-47c9-924a-fd038a206791/7dfce8f1-0c22-480c-91d4-3ffb0e2b2dff"
-					(reference "#PWR073")
-					(unit 1)
-				)
 			)
 		)
@@
 					(unit 1)
 				)
-				(path "/9003ce10-3354-47c9-924a-fd038a206791/7dfce8f1-0c22-480c-91d4-3ffb0e2b2dff"
-					(reference "#PWR068")
-					(unit 1)
-				)
 			)
 		)
@@
 					(unit 1)
 				)
-				(path "/9003ce10-3354-47c9-924a-fd038a206791/7dfce8f1-0c22-480c-91d4-3ffb0e2b2dff"
-					(reference "JP10")
-					(unit 1)
-				)
 			)
 		)
@@
 					(unit 1)
 				)
-				(path "/9003ce10-3354-47c9-924a-fd038a206791/7dfce8f1-0c22-480c-91d4-3ffb0e2b2dff"
-					(reference "#PWR063")
-					(unit 1)
-				)
 			)
 		)
@@
 					(unit 1)
 				)
-				(path "/9003ce10-3354-47c9-924a-fd038a206791/7dfce8f1-0c22-480c-91d4-3ffb0e2b2dff"
-					(reference "U3")
-					(unit 1)
-				)
 			)
 		)
@@
 					(unit 1)
 				)
-				(path "/9003ce10-3354-47c9-924a-fd038a206791/7dfce8f1-0c22-480c-91d4-3ffb0e2b2dff"
-					(reference "#PWR061")
+			)
+		)
+	)
+	(symbol
+		(lib_id "power:+3V3")
+		(at 204.47 40.64 90)
+		(unit 1)
+		(exclude_from_sim no)
+		(in_bom yes)
+		(on_board yes)
+		(dnp no)
+		(fields_autoplaced yes)
+		(property "Reference" "#PWR064"
+			(at 208.28 40.64 0)
+			(effects
+				(font
+					(size 1.27 1.27)
+				)
+				(hide yes)
+			)
+		)
+		(property "Value" "+3V3"
+			(at 200.66 40.6399 90)
+			(effects
+				(font
+					(size 1.27 1.27)
+				)
+				(justify left)
+			)
+		)
+		(property "Footprint" ""
+			(at 204.47 40.64 0)
+			(effects
+				(font
+					(size 1.27 1.27)
+				)
+				(hide yes)
+			)
+		)
+		(property "Datasheet" ""
+			(at 204.47 40.64 0)
+			(effects
+				(font
+					(size 1.27 1.27)
+				)
+				(hide yes)
+			)
+		)
+		(property "Description" "Power symbol creates a global label with name \"+3V3\""
+			(at 204.47 40.64 0)
+			(effects
+				(font
+					(size 1.27 1.27)
+				)
+				(hide yes)
+			)
+		)
+		(pin "1"
+		)
+		(instances
+			(project "LV_Regulator"
+				(path "/9003ce10-3354-47c9-924a-fd038a206791/7dabe8d0-f22d-4d1e-a460-c5fc9599efb1"
+					(reference "#PWR064")
 					(unit 1)
 				)
@@
 					(unit 1)
 				)
-				(path "/9003ce10-3354-47c9-924a-fd038a206791/7dfce8f1-0c22-480c-91d4-3ffb0e2b2dff"
-					(reference "#PWR071")
-					(unit 1)
-				)
 			)
 		)
@@
 					(unit 1)
 				)
-				(path "/9003ce10-3354-47c9-924a-fd038a206791/7dfce8f1-0c22-480c-91d4-3ffb0e2b2dff"
-					(reference "C26")
-					(unit 1)
-				)
 			)
 		)
@@
 					(unit 1)
 				)
-				(path "/9003ce10-3354-47c9-924a-fd038a206791/7dfce8f1-0c22-480c-91d4-3ffb0e2b2dff"
-					(reference "#PWR065")
-					(unit 1)
-				)
