File: LV_Kontrola_Main/LV_Kontrola_Start/LV_Kontrola_Start/Start_3V3_Isolation.kicad_sch (KiCad schematic)
At the start: 56 parts, among them IC10 UCC12040DVE, IC11 UCC12040DVE, IC12 UCC12040DVE, IC13 UCC12040DVE, IC14 UCC12040DVE, IC15 UCC12040DVE, IC16 UCC12040DVE, IC9 UCC12040DVE

Commit message: Folder structure changes
The folder structures were changed to comply with current FS Black Hornets GitHub repository templates. Separated out all the elements of the LV_Kontrola subsystem.
Other:
- title: LV_Kontrola_Main -> LV_Kontrola_Start
