File: LV_Kontrola_Main/LV_Kontrola_Start/LV_Kontrola_Start/Start_Con.kicad_sch (KiCad schematic)
At the start: 10 parts, among them J1 2169890001, J3 430451600, J4 430451600, J5 430450800, J6 430450400

Commit message: Folder structure changes
The folder structures were changed to comply with current FS Black Hornets GitHub repository templates. Separated out all the elements of the LV_Kontrola subsystem.
Other:
- title: LV_Kontrola_Main -> LV_Kontrola_Start
