File: LV_Kontrola_Main/LV_Kontrola_Start/LV_Kontrola_Start/start_control.kicad_sch (KiCad schematic)
At the start: 27 parts, among them J2 SWD, U1 ADM2483xRW, U2 STM32F103C8Tx, Y1 32.768kHz, Y2 8MHz

Commit message: Folder structure changes
The folder structures were changed to comply with current FS Black Hornets GitHub repository templates. Separated out all the elements of the LV_Kontrola subsystem.
Other:
- title: LV_Kontrola_Main -> LV_Kontrola_Start
