File: LV_Kontrola_Main/LV_Kontrola_Start/LV_Kontrola_Start/Start_Power.kicad_sch (KiCad schematic)
At the start: 15 parts, among them IC17 MIC29152WU, IC18 MIC29152WU

Commit message: Folder structure changes
The folder structures were changed to comply with current FS Black Hornets GitHub repository templates. Separated out all the elements of the LV_Kontrola subsystem.
Other:
- title: LV_Kontrola_Main -> LV_Kontrola_Start

Commit message: Started LV_Kontrola_Start pcb
Parts:
- IC17, IC18: footprint MIC29152WU:MIC29152WU -> KiCad1:MIC29152WU
Changed lines of the file:
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@@
 			)
 		)
-		(property "Footprint" "MIC29152WU:MIC29152WU"
+		(property "Footprint" "KiCad1:MIC29152WU"
 			(at 138.43 183.82 0)
 			(hide yes)
@@
 			)
 		)
-		(property "Footprint" "MIC29152WU:MIC29152WU"
+		(property "Footprint" "KiCad1:MIC29152WU"
 			(at 234.95 182.55 0)
 			(hide yes)
