File: LV_Regulator/LV_Regulator/mcu.kicad_sch (KiCad schematic)
At the start: 58 parts, among them J5 SWD, J6 2169890001, U2 STM32F103C8Tx, U3 25CSM04xxSN, Y1 32.768kHz, Y2 8MHz

Commit message: Fixed DRC & some other minor tweaks
Parts:
- R24: Purchase place https://eu.mouser.com/ProductDetail/Panasonic/ERA-8AEB103V?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 -> (none)
